File: kicad/ansic.kicad_pcb (KiCad board)
At the start: 2 copper layers, 100 x 97 mm, 62 parts, among them J1 AudioJack4, J2 AudioJack4, J3 Conn_01x02_Socket, SW1 SW_Push, SW10 SW_Push, SW11 SW_Push, SW12 SW_Push, SW13 SW_Push, SW14 SW_Push, SW15 SW_Push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

Commit message: move merge thumb layout matrix
Parts:
- renumbered SW20 to SW21
Connections:
- SW21 pad 1: Net-(D20-A) -> Net-(D21-A)
- SW21 pad 2: COL5 -> COL6
Routing:
- net Net-(D20-A): track 88.9 -> 53.9 mm
- net Net-(D21-A): track 76.6 -> 86.1 mm
- net COL6: track 139.0 -> 148.5 mm
- net COL5: track 142.2 -> 136.5 mm
Changed lines of the file:
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@@
 		(layer "F.Cu")
 		(at 155.625 115 90)
-		(property "Reference" "SW20"
+		(property "Reference" "SW21"
 			(at 0 0 90)
 			(layer "F.SilkS")
@@
 			(size 2.5 2.5)
 			(layers "B.Cu" "B.Mask" "B.Paste")
-			(net 26 "Net-(D20-A)")
+			(net 27 "Net-(D21-A)")
 			(pinfunction "1")
 			(pintype "passive")
@@
 			(size 2.5 2.5)
 			(layers "F.Cu" "F.Mask" "F.Paste")
-			(net 26 "Net-(D20-A)")
+			(net 27 "Net-(D21-A)")
 			(pinfunction "1")
 			(pintype "passive")
@@
 			(layers "*.Cu")
 			(remove_unused_layers no)
-			(net 26 "Net-(D20-A)")
+			(net 27 "Net-(D21-A)")
 			(pinfunction "1")
 			(pintype "passive")
@@
 			(layers "*.Cu")
 			(remove_unused_layers no)
-			(net 37 "COL5")
+			(net 38 "COL6")
 			(pinfunction "2")
 			(pintype "passive")
@@
 			(size 2.5 2.5)
 			(layers "B.Cu" "B.Mask" "B.Paste")
-			(net 37 "COL5")
+			(net 38 "COL6")
 			(pinfunction "2")
 			(pintype "passive")
@@
 			(size 2.5 2.5)
 			(layers "F.Cu" "F.Mask" "F.Paste")
-			(net 37 "COL5")
+			(net 38 "COL6")
 			(pinfunction "2")
 			(pintype "passive")
@@
 	)
 	(segment
-		(start 148.694 113.164257)
-		(end 148.694 118.306709)
-		(width 0.2)
-		(layer "B.Cu")
-		(net 26)
-	)
-	(segment
 		(start 109.25 102.5)
 		(end 110.099 103.349)
@@
 	)
 	(segment
-		(start 148.694 118.306709)
-		(end 151.038791 120.6515)
-		(width 0.2)
-		(layer "B.Cu")
-		(net 26)
-	)
-	(segment
-		(start 127.123 103.349)
-		(end 138.878743 103.349)
-		(width 0.2)
-		(layer "B.Cu")
-		(net 26)
-	)
-	(segment
 		(start 127.123 103.349)
 		(end 136.75 112.976)
@@
 	)
 	(segment
-		(start 138.878743 103.349)
-		(end 148.694 113.164257)
-		(width 0.2)
-		(layer "B.Cu")
-		(net 26)
-	)
-	(segment
 		(start 139.163791 120.6515)
 		(end 140.067 120.6515)
@@
 	)
 	(segment
-		(start 151.038791 120.6515)
-		(end 151.942 120.6515)
-		(width 0.2)
-		(layer "B.Cu")
-		(net 26)
-	)
-	(segment
 		(start 111.75 102.56)
 		(end 111.75 115)
@@
 	)
 	(segment
+		(start 153.085 122.085)
+		(end 162.585 122.085)
+		(width 0.2)
+		(layer "B.Cu")
+		(net 27)
+	)
+	(segment
 		(start 111.75 102.5)
 		(end 112.198 102.948)
@@
 	)
 	(segment
-		(start 141.21 107.915)
-		(end 153.085 107.915)
+		(start 143.364743 107.915)
+		(end 141.21 107.915)
 		(width 0.2)
 		(layer "F.Cu")
@@
 	)
 	(segment
-		(start 155.585 105.415)
-		(end 153.085 107.915)
+		(start 155.585 95.694743)
+		(end 143.364743 107.915)
 		(width 0.2)
 		(layer "F.Cu")
@@
 	(segment
 		(start 155.585 93.46)
-		(end 155.585 105.415)
+		(end 155.585 95.694743)
 		(width 0.2)
 		(layer "F.Cu")
@@
 		(width 0.2)
 		(layer "F.Cu")
+		(net 38)
+	)
+	(segment
+		(start 153.085 107.915)
+		(end 162.585 107.915)
+		(width 0.2)
+		(layer "F.Cu")

Commit message: fix confusing legend of silkscreen
Other:
- board text added: "FACE DOWN module component side"
- board text removed: "FACE DOWN shield component side"
Changed lines of the file:
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@@
 		(layer "Edge.Cuts")
 	)
-	(gr_text "FACE DOWN shield component side"
+	(gr_text "FACE DOWN module component side"
 		(at 92.5 48 0)
 		(layer "F.SilkS")
@@
 		)
 	)
-	(gr_text "FACE DOWN shield component side"
+	(gr_text "FACE DOWN module component side"
 		(at 92.5 48 -0)
 		(layer "B.SilkS")
